File: schematics/v2/main.sch (EAGLE design)
At the start: 15 parts, among them IC1 MEGA8-P, Q1 BC548

Commit message: Updating schematics for v2
Parts:
- removed X1: (no value), con-wago-500:W237-102
- added C1: 100n, rcl:C-EU025-025X050
- added C2: 47u, rcl:CPOL-EUE2.5-6
- added C3: 10u, rcl:CPOL-EUE2.5-6
- added D1: 1N4007, diode:DIODE-D-7.5
- added IC2: 7805T, linear:7805T
- added JP1: RS232, jumper:JP1E
- added LED2: (no value), led:LED5MM
- added R5: 330, resistor:R-EU_0204/7
Connections:
- new net N$12: LED2.C, R5.2
- new net N$13: IC1.PD1(TXD), JP1.1
- net +12V: now also C2.+, C3.+, IC2.VI
- net +5V: now also C1.1, D1.C, IC2.VO, LED2.A; no longer X1-1.KL
- net GND: now also C1.2, C2.-, C3.-, D1.A, IC2.GND, JP1.2, R5.1; no longer X1-2.KL
